Commit message: Added RECIRCULATE files and modified robot descriptions

File: kuka_agilus_support/urdf/kr10_r1100_2_macro.xacro (robot description, xacro)
@@ -158,5 +158,5 @@
       <parent link="${prefix}base_link" />
       <child link="${prefix}base_link_inertia" />
-      <origin xyz="0 0 2.0" rpy="${pi} 0 0" />
+      <origin xyz="-0.4 0 2.0" rpy="${pi} 0 0" />
     </joint>
     <joint name="${prefix}joint_1" type="revolute">
