Commit message: Added RECIRCULATE files and modified robot descriptions

File: kuka_agilus_support/urdf/kr10_r1100_2.urdf.xacro (robot description, xacro)
@@ -6,3 +6,4 @@
   <xacro:arg name="use_fake_hardware" default="false" />
   <xacro:kuka_kr10_r1100_2_robot prefix="" use_fake_hardware="$(arg use_fake_hardware)"/>
+<xacro:include filename="$(find kuka_agilus_support)/urdf/recirculate.xacro"/>
 </robot>

File: kuka_agilus_support/urdf/kr10_r1100_2_macro.xacro (robot description, xacro)
@@ -158,5 +158,5 @@
       <parent link="${prefix}base_link" />
       <child link="${prefix}base_link_inertia" />
-      <origin xyz="0 0 0" rpy="0 0 0" />
+      <origin xyz="0 0 2.0" rpy="${pi} 0 0" />
     </joint>
     <joint name="${prefix}joint_1" type="revolute">

Commit message: added linear track config

File: kuka_agilus_support/urdf/kr10_r1100_2.urdf.xacro (robot description, xacro)
@@ -1,9 +1,22 @@
 <?xml version="1.0"?>
-<robot xmlns:xacro="http://www.ros.org/wiki/xacro" name="kr10_r1100_2">
+<robot xmlns:xacro="http://www.ros.org/wiki/xacro" name="kr10_r1100_2_ext_axis">
   <!-- Import urdf file  -->
+  <xacro:include filename="$(find kuka_agilus_support)/urdf/kl100_linear_axis.xacro"/>
   <xacro:include filename="$(find kuka_agilus_support)/urdf/kr10_r1100_2_macro.xacro"/>
   <!-- Read additional arguments  -->
   <xacro:arg name="use_fake_hardware" default="false" />
+<!--xacro:include filename="$(find kuka_agilus_support)/urdf/recirculate.xacro"/-->
+  <link name="world" />
+  <joint name="world_joint" type="fixed">
+            <parent link="world" />
+            <child link="kl100_frame" />
+            <origin xyz="0.0 0.0 0.0" rpy="0.0 0.0 0.0" />
+        </joint>
+  <xacro:kl100_linear_axis prefix=""/>
+        <joint name="attachment_joint" type="fixed">
+            <parent link="axis7" />
+            <child link="base_link" />
+            <origin xyz="0.0 0.0 0.0" rpy="0 0 0" />
+        </joint>
   <xacro:kuka_kr10_r1100_2_robot prefix="" use_fake_hardware="$(arg use_fake_hardware)"/>
-<xacro:include filename="$(find kuka_agilus_support)/urdf/recirculate.xacro"/>
 </robot>

File: kuka_agilus_support/urdf/kr10_r1100_2_macro.xacro (robot description, xacro)
@@ -158,5 +158,5 @@
       <parent link="${prefix}base_link" />
       <child link="${prefix}base_link_inertia" />
-      <origin xyz="-0.4 0 2.0" rpy="${pi} 0 0" />
+      <origin xyz="0.08 0.1 0" rpy="${pi} 0 ${-pi/2}" />
     </joint>
     <joint name="${prefix}joint_1" type="revolute">
